Commit message: Update Robot.urdf
Added joint limit for Joint 2 (NodeFL - NodeFR)

File: Robot.urdf (robot description, URDF)
Before this commit: robot Robot, 12 links, 11 joints
Joints:
- joint NodeFRtoFL: limit lower=0 upper=0 effort=1.667 velocity=0 -> lower=-1 upper=1 effort=1.667 velocity=0

Commit message: Updates
Updates to URDF, code, currently set up for transverse movement

File: Robot.urdf (robot description, URDF)
Before this commit: robot Robot, 12 links, 11 joints
Joints:
- joint NodeBLtoFL: limit lower=0 upper=0 effort=1.667 velocity=0 -> lower=-1 upper=1 effort=1.667 velocity=0
- joint NodeBRtoFR: limit lower=0 upper=0 effort=1.667 velocity=0 -> lower=-1 upper=1 effort=1.667 velocity=0

Commit message: Fixed the origin of bottom legs

File: Robot.urdf (robot description, URDF)
Before this commit: robot Robot, 12 links, 11 joints
Links:
- link LegBLbottom: mass 0.18815 -> 0.18815446532302
- link LegBLtop: mass 0.41495 -> 0.414951621421335
- link LegBRbottom: mass 0.18815 -> 0.188154465331508
- link LegBRtop: mass 0.41495 -> 0.414951621421334
- link LegFLbottom: mass 0.18815 -> 0.188154465332503
- link LegFLtop: mass 0.41495 -> 0.414951621421333
- link LegFRbottom: mass 0.18815 -> 0.188154465333161
- link LegFRtop: mass 0.41495 -> 0.414951621421329
- link NodeBL: mass 0 -> 3.81292986220067
- link NodeBR: mass 3.796 -> 3.79597569263433
- link NodeFL: mass 3.5578 -> 3.55778654478529
- link NodeFR: mass 3.5744 -> 3.57441614761339
Joints:
- joint LegBLbottomJoint: axis 0 0 -1 -> 0 -1 0; origin xyz=0 0 0.004743 rpy=3.1416 0 1.5536 -> xyz=0.0259811300575554 -0.244963993367846 0.0392430236363058 rpy=-1.5707963267949 0 -0.319261233206899
- joint LegBLtopJoint: axis 0 0 1 -> 0 0 -1; origin xyz=0.30766 -0.010974 9.8262E-05 rpy=-1.5708 1.0174 -1.5708 -> xyz=0.307656976363671 -0.0109741059783897 9.82624883940075E-05 rpy=-1.5707963267949 1.01739293400464 -1.5707963267949
- joint LegBRbottomJoint: axis 0 0 -1 -> 0 1 0; origin xyz=0 0 -0.004743 rpy=3.1416 0 1.6741 -> xyz=-0.0133692926627684 -0.242601325331272 -0.0392430236362956 rpy=-1.57079632679485 0 -0.48442729599235
- joint LegBRtopJoint: axis 0 0 1 -> 0 0 -1; origin xyz=-0.0042984 -0.19589 0.049227 rpy=-2.7873 -0.14095 -1.2078 -> xyz=-0.00429840728729508 -0.195893220384569 0.0492268311937279 rpy=-2.78731505033292 -0.140945170035096 -1.20783082058472
- joint LegFLbottomJoint: axis 1 0 0 -> 0 1 0; origin xyz=0 0 0.004743 rpy=0.010584 -1.5708 0.010584 -> xyz=0.0349508441723456 -0.243845885053306 0.0392430236363057 rpy=1.5707963267949 0 2.8590275181257
- joint LegFLtopJoint: axis 0 0 1 -> 0 0 -1; origin xyz=0.00085062 0.0033885 0.050662 rpy=1.5708 0.5901 1.5708 -> xyz=0.000850617108481061 0.00338851971521293 0.050662338857125 rpy=1.5707963267949 0.59009949053307 1.5707963267949
- joint LegFRbottomJoint: axis -1 0 0 -> 0 1 0; origin xyz=0 0 -0.004743 rpy=3.0317 1.5708 0 -> xyz=0.0489781894022524 -0.237981675768681 -0.0392430236363144 rpy=-1.57079632679487 0 -0.22640240015338
- joint LegFRtopJoint: axis 0 0 1 -> 0 0 -1; origin xyz=0.0067323 -0.31401 -0.046653 rpy=-1.5708 0.75396 0 -> xyz=0.00673229574135756 -0.314006976363694 -0.0466526058184806 rpy=-1.5707963267949 0.753964187321215 0
- joint NodeBLtoFL: limit lower=-1 upper=1 effort=1.667 velocity=0 -> lower=0 upper=0 effort=1.667 velocity=0; origin xyz=-0.30641 0.40561 0.046076 rpy=1.5708 0 0 -> xyz=-0.306406359255212 0.40560642659738 0.046075935941584 rpy=1.5707963267949 0 0
- joint NodeBRtoFR: limit lower=-1 upper=1 effort=1.667 velocity=0 -> lower=0 upper=0 effort=1.667 velocity=0; origin xyz=0.042552 -0.2667 -0.24704 rpy=1.507 -0.15828 0.38525 -> xyz=0.0425516484371528 -0.2667 -0.247043441975824 rpy=1.50696525699484 -0.158283867014591 0.385246744254906
- joint NodeFRtoFL: limit lower=-1 upper=1 effort=1.667 velocity=0 -> lower=0 upper=0 effort=1.667 velocity=0; origin xyz=-0.22314 -0.041066 0.049378 rpy=3.1416 1.4002 1.5708 -> xyz=-0.223136085546314 -0.0410663380019626 0.049377935941584 rpy=3.14159265358979 1.400226413165 1.5707963267949

Commit message: URDF update

File: Robot.urdf (robot description, URDF)
Before this commit: robot Robot, 12 links, 11 joints
Joints:
- joint NodeBLtoFL: limit lower=0 upper=0 effort=1.667 velocity=0 -> lower=-1 upper=1 effort=1.667 velocity=0
- joint NodeBRtoFR: limit lower=0 upper=0 effort=1.667 velocity=0 -> lower=-1 upper=1 effort=1.667 velocity=0
- joint NodeFRtoFL: limit lower=0 upper=0 effort=1.667 velocity=0 -> lower=-1 upper=1 effort=1.667 velocity=0

Commit message: mass update

File: Robot.urdf (robot description, URDF)
Before this commit: robot Robot, 12 links, 11 joints
Links:
- link LegBLbottom: mass 0.18815446532302 -> 60
- link LegBLtop: mass 0.414951621421335 -> 60
- link LegBRbottom: mass 0.188154465331508 -> 60
- link LegBRtop: mass 0.414951621421334 -> 60
- link LegFLbottom: mass 0.188154465332503 -> 60
- link LegFLtop: mass 0.414951621421333 -> 60
- link LegFRbottom: mass 0.188154465333161 -> 60
- link LegFRtop: mass 0.414951621421329 -> 60
- link NodeBL: mass 3.81292986220067 -> 70
- link NodeBR: mass 3.79597569263433 -> 70
- link NodeFL: mass 3.55778654478529 -> 70
- link NodeFR: mass 3.57441614761339 -> 70

Commit message: limits

File: Robot.urdf (robot description, URDF)
Before this commit: robot Robot, 12 links, 11 joints
Joints:
- joint LegBLbottomJoint: limit lower=-1.5 upper=1.5 effort=1.667 velocity=6.25 -> lower=0 upper=0.5 effort=1.667 velocity=6.25
- joint NodeBLtoFL: limit lower=-1 upper=1 effort=1.667 velocity=0 -> lower=0 upper=0.5 effort=1.667 velocity=0
- joint NodeBRtoFR: limit lower=-1 upper=1 effort=1.667 velocity=0 -> lower=0 upper=0.5 effort=1.667 velocity=0
- joint NodeFRtoFL: limit lower=-1 upper=1 effort=1.667 velocity=0 -> lower=0 upper=.5 effort=1.667 velocity=0

Commit message: random and hill climber ready

File: Robot.urdf (robot description, URDF)
Before this commit: robot Robot, 12 links, 11 joints
Links:
- link LegBLbottom: mass 60 -> 600
- link LegBLtop: mass 60 -> 600
- link LegBRbottom: mass 60 -> 600
- link LegBRtop: mass 60 -> 600
- link LegFLbottom: mass 60 -> 600
- link LegFLtop: mass 60 -> 600
- link LegFRbottom: mass 60 -> 600
- link LegFRtop: mass 60 -> 600
- link NodeBL: mass 70 -> 700
- link NodeBR: mass 70 -> 700
- link NodeFL: mass 70 -> 700
- link NodeFR: mass 70 -> 700
Joints:
- joint LegBLbottomJoint: limit lower=0 upper=0.5 effort=1.667 velocity=6.25 -> lower=-0.05 upper=0.05 effort=1.667 velocity=6.25
- joint LegBLtopJoint: limit lower=-1.5 upper=1.5 effort=1.667 velocity=6.25 -> lower=-1.25 upper=1.25 effort=1.667 velocity=6.25
- joint LegBRbottomJoint: limit lower=-1.5 upper=1.5 effort=1.667 velocity=6.25 -> lower=-1.25 upper=1.25 effort=1.667 velocity=6.25
- joint LegBRtopJoint: limit lower=-1.5 upper=1.5 effort=1.667 velocity=6.25 -> lower=-1.25 upper=1.25 effort=1.667 velocity=6.25
- joint LegFLbottomJoint: limit lower=-1.5 upper=1.5 effort=1.667 velocity=6.25 -> lower=-1.25 upper=1.25 effort=1.667 velocity=6.25
- joint LegFLtopJoint: limit lower=-1.5 upper=1.5 effort=1.667 velocity=6.25 -> lower=-1.25 upper=1.25 effort=1.667 velocity=6.25
- joint LegFRbottomJoint: limit lower=-1.5 upper=1.5 effort=1.667 velocity=6.25 -> lower=-1.25 upper=1.25 effort=1.667 velocity=6.25
- joint LegFRtopJoint: limit lower=-1.5 upper=1.5 effort=1.667 velocity=6.25 -> lower=-1.25 upper=1.25 effort=1.667 velocity=6.25
- joint NodeBLtoFL: limit lower=0 upper=0.5 effort=1.667 velocity=0 -> lower=-.05 upper=.05 effort=1.667 velocity=0
- joint NodeBRtoFR: limit lower=0 upper=0.5 effort=1.667 velocity=0 -> lower=-0.05 upper=0.05 effort=1.667 velocity=0
- joint NodeFRtoFL: limit lower=0 upper=.5 effort=1.667 velocity=0 -> lower=-0.05 upper=0.05 effort=1.667 velocity=0
